File: final_project/final_project.sch (KiCad schematic (older format))
At the start: 60 parts, among them J1 USB_microB_2040002-1, J2 Arduino_ICSP, J3 Conn_01x06_Male, U1 FT232RQ, U10 MAX14870, U2 MCP1702T-5002E_CB, U3 TPS2113ADRBR, U4 ATMEGA328PB-MNR, U5 RN4871, U6 ISM330DLC, U7 MAX14870, U8 MAX14870, U9 MAX14870, Y1 Crystal

Commit message: add logic level converter
Parts:
- removed R11: 4.7K, Resistor_SMD:R_0603_1608Metric, symbol Device:R
- removed S2: SW, Button_Switch_SMD:SW_SPST_B3U-1000P, symbol final_project-rescue:SW-final_project
- added U11: TXB0108_RGYR, symbol final_project-rescue:TXB0108_RGYR
- R17, R19, R20: value 330 -> 1k
Connections:
- net GNDorVdd is gone; now on net GND: U6.2 (SDX), U6.3 (SCX)
- net +3V3: now also U11.2 (V_cca); no longer D5.2 (A), D7.2 (A), D8.2 (A)
- net +5V: now also D5.2 (A), D7.2 (A), D8.2 (A), U11.10 (OE), U11.19 (V_ccb)
- net A5: no longer U4.28 (PC5/ADC5/SCL), U6.13 (SCC)
- net GND: now also U11.11 (GND)
- net logic2_3: now reaches U5.10 (-RST)
- net logic2_3: now also U11.3 (A2)
- net A0 renamed logic1_3
- net logic1_3: now also U11.1 (A1); no longer U4.23 (PC0/ADC0)
- net A1 renamed logic6_3
- net logic6_3: now also U11.14 (B6), U11.7 (A6); no longer U4.24 (PC1/ADC1)
- net A4 renamed logic8_3
- net logic8_3: now also U11.9 (A8); no longer U4.27 (PC4/ADC4/SDA)
- net A7: no longer names the net of U4.22 (ADC7)
- net D3: no longer names the net of U5.11 (P0_0)
- net D3: no longer U4.1 (PD3/INT1)
- net D4: no longer names the net of U4.2 (PD4/XCK/T0)
- net D4: no longer U5.9 (P3_6)
- net D5 renamed logic3_3
- net logic3_3: now also U11.4 (A3); no longer U4.9 (PD5/T1)
- net D6 renamed logic4_3
- net logic4_3: now also U11.5 (A4); no longer U4.10 (PD6/AIN0)
- net D8 renamed logic5_3
- net logic5_3: now also U11.6 (A5); no longer U4.12 (PB0/ICP)
- new net logic1_5: U11.20 (B1), U4.23 (PC0/ADC0)
- new net logic2_5: U11.18 (B2), U4.1 (PD3/INT1)
- new net logic3_5: U11.17 (B3), U4.9 (PD5/T1)
- new net logic4_5: U11.16 (B4), U4.10 (PD6/AIN0)
- new net logic5_5: U11.15 (B5), U4.12 (PB0/ICP)
- new net logic6_5: U4.24 (PC1/ADC1)
- new net logic7_3: U11.8 (A7), U6.13 (SCC)
- new net logic7_5: U11.13 (B7), U4.28 (PC5/ADC5/SCL)
- new net logic8_5: U11.12 (B8), U4.27 (PC4/ADC4/SDA)
- no-connect marks 28 -> 32
Other:
- moved on the sheet: C12, C14, D8, R20, U6

Commit message: adding power and motor connectors (symbols and footprints)
Parts:
- added U? (x2): 8_pin_screw_terminal, symbol final_project-rescue:8_pin_screw_terminal
- added U?: 2_pin_screw_terminal, symbol final_project-rescue:2_pin_screw_terminal
Connections:
- net +BATT: now also U?.1 (m1a), U?.3 (m2a), U?.5 (m3a), U?.7 (m4a)
- net GND: now also U?.2 (GND), U?.2 (m1b), U?.4 (m2b), U?.6 (m3b), U?.8 (m4b)
- net VIN: now also U?.1 (3.7V)
- net motor1a: now also U?.1 (m1a)
- net motor1b: now also U?.2 (m1b)
- net motor2a: now also U?.3 (m2a)
- net motor2b: now also U?.4 (m2b)
- net motor3a: now also U?.5 (m3a)
- net motor3b: now also U?.6 (m3b)
- net motor4a: now also U?.7 (m4a)
- net motor4b: now also U?.8 (m4b)
Changed lines of the file:
@@
 $EndComp
 NoConn ~ 10900 7600
+$Comp
+L final_project-rescue:8_pin_screw_terminal U?
+U 1 1 5CAE560A
+P 15850 2950
+F 0 "U?" H 15929 2996 50  0000 L CNN
+F 1 "8_pin_screw_terminal" H 15929 2905 50  0000 L CNN
+F 2 "" H 15850 2950 50  0001 C CNN
+F 3 "" H 15850 2950 50  0001 C CNN
+	1    15850 2950
+	1    0    0    -1
+$EndComp
+Text Label 15350 2750 0    50   ~ 0
+motor1a
+Text Label 15350 2800 0    50   ~ 0
+motor1b
+Text Label 15350 2850 0    50   ~ 0
+motor2a
+Text Label 15350 2900 0    50   ~ 0
+motor2b
+Text Label 15350 3000 0    50   ~ 0
+motor3a
+Text Label 15350 3050 0    50   ~ 0
+motor3b
+Text Label 15350 3100 0    50   ~ 0
+motor4a
+Text Label 15350 3150 0    50   ~ 0
+motor4b
+Wire Wire Line
+	15350 2750 15700 2750
+Wire Wire Line
+	15700 2800 15350 2800
+Wire Wire Line
+	15350 2850 15700 2850
+Wire Wire Line
+	15350 2900 15700 2900
+Wire Wire Line
+	15350 3000 15700 3000
+Wire Wire Line
+	15700 3050 15350 3050
+Wire Wire Line
+	15350 3100 15700 3100
+Wire Wire Line
+	15350 3150 15700 3150
+$Comp
+L final_project-rescue:8_pin_screw_terminal U?
+U 1 1 5CB47892
+P 10300 2800
+F 0 "U?" H 10379 2846 50  0000 L CNN
+F 1 "8_pin_screw_terminal" H 10379 2755 50  0000 L CNN
+F 2 "" H 10300 2800 50  0001 C CNN
+F 3 "" H 10300 2800 50  0001 C CNN
+	1    10300 2800
+	1    0    0    -1
+$EndComp
+$Comp
+L power:+BATT #PWR?
+U 1 1 5CB48118
+P 10000 2600
+F 0 "#PWR?" H 10000 2450 50  0001 C CNN
+F 1 "+BATT" H 10015 2773 50  0000 C CNN
+F 2 "" H 10000 2600 50  0001 C CNN
+F 3 "" H 10000 2600 50  0001 C CNN
+	1    10000 2600
+	1    0    0    -1
+$EndComp
+$Comp
+L power:GND #PWR?
+U 1 1 5CB481BB
+P 9850 3000
+F 0 "#PWR?" H 9850 2750 50  0001 C CNN
+F 1 "GND" H 9855 2827 50  0000 C CNN
+F 2 "" H 9850 3000 50  0001 C CNN
+F 3 "" H 9850 3000 50  0001 C CNN
+	1    9850 3000
+	1    0    0    -1
+$EndComp
+Wire Wire Line
+	10150 2600 10000 2600
+Wire Wire Line
+	10150 2700 10000 2700
+Wire Wire Line
+	10000 2700 10000 2600
+Connection ~ 10000 2600
+Wire Wire Line
+	10150 2850 10000 2850
+Wire Wire Line
+	10000 2850 10000 2700
+Connection ~ 10000 2700
+Wire Wire Line
+	10150 2950 10000 2950
+Wire Wire Line
+	10000 2950 10000 2850
+Connection ~ 10000 2850
+Wire Wire Line
+	10150 2650 9850 2650
+Wire Wire Line
+	9850 2650 9850 2750
+Wire Wire Line
+	10150 2750 9850 2750
+Connection ~ 9850 2750
+Wire Wire Line
+	9850 2750 9850 2900
+Wire Wire Line
+	10150 2900 9850 2900
+Connection ~ 9850 2900
+Wire Wire Line
+	9850 2900 9850 3000
+Wire Wire Line
+	10150 3000 9850 3000
+Connection ~ 9850 3000
+$Comp
+L final_project-rescue:2_pin_screw_terminal U?
+U 1 1 5CBB3A54
+P 2200 1950
+F 0 "U?" H 2328 1996 50  0000 L CNN
+F 1 "2_pin_screw_terminal" H 2328 1905 50  0000 L CNN
+F 2 "" H 2200 1950 50  0001 C CNN
+F 3 "" H 2200 1950 50  0001 C CNN
+	1    2200 1950
+	1    0    0    -1
+$EndComp
+Text Label 1850 1850 0    50   ~ 0
+VIN
+$Comp
+L power:GND #PWR?
+U 1 1 5CBB3C6A
+P 1900 2200
+F 0 "#PWR?" H 1900 1950 50  0001 C CNN
+F 1 "GND" H 1905 2027 50  0000 C CNN
+F 2 "" H 1900 2200 50  0001 C CNN
+F 3 "" H 1900 2200 50  0001 C CNN
+	1    1900 2200
+	1    0    0    -1
+$EndComp
+Wire Wire Line
+	2000 2050 1900 2050
+Wire Wire Line
+	1900 2050 1900 2200
+Wire Wire Line
+	2000 1850 1850 1850
 $EndSCHEMATC
