File: final_project/final_project.sch (KiCad schematic (older format))
At the start: 62 parts, among them J1 USB_microB_2040002-1, J2 Arduino_ICSP, J3 Conn_01x06_Male, U1 FT232RQ, U10 MAX14870, U11 TXB0108_RGYR, U2 MCP1702T-5002E_CB, U3 TPS2113ADRBR, U4 ATMEGA328PB-MNR, U5 RN4871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

Commit message: new things
Parts:
- J3: footprint (none) -> Connector_PinHeader_2.54mm:PinHeader_1x06_P2.54mm_Vertical
- U12: renamed from U?; footprint (none) -> final:2_pin_screw
- U13, U14: renamed from U?; footprint (none) -> final:8_pin_screw
- U5: footprint (none) -> final:RN4871
- U6: footprint (none) -> final:ISM330DLC
Changed lines of the file:
@@
 F 0 "U6" H 4200 9350 50  0000 C CNN
 F 1 "ISM330DLC" H 4200 9250 50  0000 C CNN
-F 2 "" H 4150 7800 50  0001 C CNN
+F 2 "final:ISM330DLC" H 4150 7800 50  0001 C CNN
 F 3 "" H 4150 7800 50  0001 C CNN
 	1    4150 8400
@@
 F 0 "U5" H 13050 7615 50  0000 C CNN
 F 1 "RN4871" H 13050 7524 50  0000 C CNN
-F 2 "" H 13050 7650 50  0001 C CNN
+F 2 "final:RN4871" H 13050 7650 50  0001 C CNN
 F 3 "" H 13050 7650 50  0001 C CNN
 	1    13050 6800
@@
 F 0 "J3" H 1706 7128 50  0000 C CNN
 F 1 "Conn_01x06_Male" H 1706 7037 50  0000 C CNN
-F 2 "" H 1600 6750 50  0001 C CNN
+F 2 "Connector_PinHeader_2.54mm:PinHeader_1x06_P2.54mm_Vertical" H 1600 6750 50  0001 C CNN
 F 3 "~" H 1600 6750 50  0001 C CNN
 	1    1600 6750
@@
 NoConn ~ 10900 7600
 $Comp
-L final_project-rescue:8_pin_screw_terminal U?
+L final_project-rescue:8_pin_screw_terminal U14
 U 1 1 5CAE560A
 P 15850 2950
-F 0 "U?" H 15929 2996 50  0000 L CNN
+F 0 "U14" H 15929 2996 50  0000 L CNN
 F 1 "8_pin_screw_terminal" H 15929 2905 50  0000 L CNN
-F 2 "" H 15850 2950 50  0001 C CNN
+F 2 "final:8_pin_screw" H 15850 2950 50  0001 C CNN
 F 3 "" H 15850 2950 50  0001 C CNN
 	1    15850 2950
@@
 	15350 3150 15700 3150
 $Comp
-L final_project-rescue:8_pin_screw_terminal U?
+L final_project-rescue:8_pin_screw_terminal U13
 U 1 1 5CB47892
 P 10300 2800
-F 0 "U?" H 10379 2846 50  0000 L CNN
+F 0 "U13" H 10379 2846 50  0000 L CNN
 F 1 "8_pin_screw_terminal" H 10379 2755 50  0000 L CNN
-F 2 "" H 10300 2800 50  0001 C CNN
+F 2 "final:8_pin_screw" H 10300 2800 50  0001 C CNN
 F 3 "" H 10300 2800 50  0001 C CNN
 	1    10300 2800
@@
 $EndComp
 $Comp
-L power:+BATT #PWR?
+L power:+BATT #PWR0142
 U 1 1 5CB48118
 P 10000 2600
-F 0 "#PWR?" H 10000 2450 50  0001 C CNN
+F 0 "#PWR0142" H 10000 2450 50  0001 C CNN
 F 1 "+BATT" H 10015 2773 50  0000 C CNN
 F 2 "" H 10000 2600 50  0001 C CNN
@@
 $EndComp
 $Comp
-L power:GND #PWR?
+L power:GND #PWR0143
 U 1 1 5CB481BB
 P 9850 3000
-F 0 "#PWR?" H 9850 2750 50  0001 C CNN
+F 0 "#PWR0143" H 9850 2750 50  0001 C CNN
 F 1 "GND" H 9855 2827 50  0000 C CNN
 F 2 "" H 9850 3000 50  0001 C CNN
@@
 Connection ~ 9850 3000
 $Comp
-L final_project-rescue:2_pin_screw_terminal U?
+L final_project-rescue:2_pin_screw_terminal U12
 U 1 1 5CBB3A54
 P 2200 1950
-F 0 "U?" H 2328 1996 50  0000 L CNN
+F 0 "U12" H 2328 1996 50  0000 L CNN
 F 1 "2_pin_screw_terminal" H 2328 1905 50  0000 L CNN
-F 2 "" H 2200 1950 50  0001 C CNN
+F 2 "final:2_pin_screw" H 2200 1950 50  0001 C CNN
 F 3 "" H 2200 1950 50  0001 C CNN
 	1    2200 1950
@@
 VIN
 $Comp
-L power:GND #PWR?
+L power:GND #PWR0144
 U 1 1 5CBB3C6A
 P 1900 2200
-F 0 "#PWR?" H 1900 1950 50  0001 C CNN
+F 0 "#PWR0144" H 1900 1950 50  0001 C CNN
 F 1 "GND" H 1905 2027 50  0000 C CNN
 F 2 "" H 1900 2200 50  0001 C CNN

Commit message: adding footprint for motor controllers and attatching some other footprints
Parts:
- U10, U7, U8, U9: footprint (none) -> Package_DFN_QFN:DFN-12-1EP_3x3mm_P0.5mm_EP2.05x2.86mm
Changed lines of the file:
@@
 F 0 "U7" H 12325 2625 50  0000 C CNN
 F 1 "MAX14870" H 12325 2534 50  0000 C CNN
-F 2 "" H 12300 2200 50  0001 C CNN
+F 2 "Package_DFN_QFN:DFN-12-1EP_3x3mm_P0.5mm_EP2.05x2.86mm" H 12300 2200 50  0001 C CNN
 F 3 "" H 12300 2200 50  0001 C CNN
 	1    12300 2200
@@
 F 0 "U9" H 14175 2625 50  0000 C CNN
 F 1 "MAX14870" H 14175 2534 50  0000 C CNN
-F 2 "" H 14150 2200 50  0001 C CNN
+F 2 "Package_DFN_QFN:DFN-12-1EP_3x3mm_P0.5mm_EP2.05x2.86mm" H 14150 2200 50  0001 C CNN
 F 3 "" H 14150 2200 50  0001 C CNN
 	1    14150 2200
@@
 F 0 "U8" H 12325 4725 50  0000 C CNN
 F 1 "MAX14870" H 12325 4634 50  0000 C CNN
-F 2 "" H 12300 4300 50  0001 C CNN
+F 2 "Package_DFN_QFN:DFN-12-1EP_3x3mm_P0.5mm_EP2.05x2.86mm" H 12300 4300 50  0001 C CNN
 F 3 "" H 12300 4300 50  0001 C CNN
 	1    12300 4300
@@
 F 0 "U10" H 14175 4725 50  0000 C CNN
 F 1 "MAX14870" H 14175 4634 50  0000 C CNN
-F 2 "" H 14150 4300 50  0001 C CNN
+F 2 "Package_DFN_QFN:DFN-12-1EP_3x3mm_P0.5mm_EP2.05x2.86mm" H 14150 4300 50  0001 C CNN
 F 3 "" H 14150 4300 50  0001 C CNN
 	1    14150 4300

Commit message: TDFN's
Parts:
- U10, U7, U8, U9: footprint Package_DFN_QFN:DFN-12-1EP_3x3mm_P0.5mm_EP2.05x2.86mm -> final:TDFN-12-1EP_3x3
Changed lines of the file:
@@
 F 0 "U7" H 12325 2625 50  0000 C CNN
 F 1 "MAX14870" H 12325 2534 50  0000 C CNN
-F 2 "Package_DFN_QFN:DFN-12-1EP_3x3mm_P0.5mm_EP2.05x2.86mm" H 12300 2200 50  0001 C CNN
+F 2 "final:TDFN-12-1EP_3x3" H 12300 2200 50  0001 C CNN
 F 3 "" H 12300 2200 50  0001 C CNN
 	1    12300 2200
@@
 F 0 "U9" H 14175 2625 50  0000 C CNN
 F 1 "MAX14870" H 14175 2534 50  0000 C CNN
-F 2 "Package_DFN_QFN:DFN-12-1EP_3x3mm_P0.5mm_EP2.05x2.86mm" H 14150 2200 50  0001 C CNN
+F 2 "final:TDFN-12-1EP_3x3" H 14150 2200 50  0001 C CNN
 F 3 "" H 14150 2200 50  0001 C CNN
 	1    14150 2200
@@
 F 0 "U8" H 12325 4725 50  0000 C CNN
 F 1 "MAX14870" H 12325 4634 50  0000 C CNN
-F 2 "Package_DFN_QFN:DFN-12-1EP_3x3mm_P0.5mm_EP2.05x2.86mm" H 12300 4300 50  0001 C CNN
+F 2 "final:TDFN-12-1EP_3x3" H 12300 4300 50  0001 C CNN
 F 3 "" H 12300 4300 50  0001 C CNN
 	1    12300 4300
@@
 F 0 "U10" H 14175 4725 50  0000 C CNN
 F 1 "MAX14870" H 14175 4634 50  0000 C CNN
-F 2 "Package_DFN_QFN:DFN-12-1EP_3x3mm_P0.5mm_EP2.05x2.86mm" H 14150 4300 50  0001 C CNN
+F 2 "final:TDFN-12-1EP_3x3" H 14150 4300 50  0001 C CNN
 F 3 "" H 14150 4300 50  0001 C CNN
 	1    14150 4300

Commit message: first pass layout
Parts:
- removed U11: TXB0108_RGYR, symbol final_project-rescue:TXB0108_RGYR
- added U11: TXB0108_DQS, final:USON-20_2x4mm_P0.4mm, symbol final_project-rescue:TXB0108_DQS
Connections:
- net +3V3: now also U11.5 (V_cca)
- net +5V: now also U11.16 (V_ccb), U11.6 (OE)
- net GND: now also U11.15 (GND)
- net logic1_3: now also U11.1 (A1)
- net logic1_5: now also U11.20 (B1)
- net logic2_3: now also U11.2 (A2)
- net logic2_5: now also U11.19 (B2)
- net logic3_3: now also U11.3 (A3)
- net logic3_5: now also U11.18 (B3)
- net logic4_3: now also U11.4 (A4)
- net logic4_5: now also U11.17 (B4)
- net logic5_3: now also U11.7 (A5)
- net logic5_5: now also U11.14 (B5)
- net logic6_3: now also U11.8 (A6)
- net logic6_5: now also U11.13 (B6)
- net logic7_3: now also U11.9 (A7)
- net logic7_5: now also U11.12 (B7)
- net logic8_3: now also U11.10 (A8)
- net logic8_5: now also U11.11 (B8)
Changed lines of the file:
@@
 encoding utf-8
 Sheet 1 1
-Title "Miniproject 3 Version A"
-Date ""
+Title "Final Project"
+Date "Spring 2019"
 Rev ""
 Comp "Olin College of Engineering"
-Comment1 ""
+Comment1 "Anne Kroo, Emma Westerhoff, Kim Winter"
 Comment2 ""
 Comment3 ""
@@
 $EndComp
 NoConn ~ 10900 5400
-$Comp
-L final_project-rescue:TXB0108_RGYR U11
-U 1 1 5CB4B187
-P 7500 9000
-F 0 "U11" H 7500 10200 50  0000 C CNN
-F 1 "TXB0108_RGYR" H 7500 10100 50  0000 C CNN
-F 2 "" H 7400 9250 50  0001 C CNN
-F 3 "" H 7400 9250 50  0001 C CNN
-	1    7500 9000
-	1    0    0    -1
-$EndComp
 Text Label 7050 8400 2    50   ~ 0
 logic1_3
@@
 logic7_5
 Text Label 7950 9150 0    50   ~ 0
-logic6_3
+logic6_5
 Text Label 7950 9000 0    50   ~ 0
 logic5_5
@@
 Wire Wire Line
 	2000 1850 1850 1850
+$Comp
+L final_project-rescue:TXB0108_DQS U11
+U 1 1 5CAFC4B6
+P 7500 9000
+F 0 "U11" H 7500 10000 50  0000 C CNN
+F 1 "TXB0108_DQS" H 7500 10100 50  0000 C CNN
+F 2 "final:USON-20_2x4mm_P0.4mm" H 7400 9250 50  0001 C CNN
+F 3 "" H 7400 9250 50  0001 C CNN
+	1    7500 9000
+	1    0    0    -1
+$EndComp
 $EndSCHEMATC

Commit message: updated layout v1
Connections:
- net +BATT: no longer U13.1 (m1a), U13.3 (m2a)
- net GND: no longer U13.6 (m3b), U13.8 (m4b)
- new net: U13.1 (m1a), U13.3 (m2a), U13.6 (m3b), U13.8 (m4b)
Changed lines of the file:
@@
 L power:+BATT #PWR0142
 U 1 1 5CB48118
-P 10000 2600
-F 0 "#PWR0142" H 10000 2450 50  0001 C CNN
-F 1 "+BATT" H 10015 2773 50  0000 C CNN
-F 2 "" H 10000 2600 50  0001 C CNN
-F 3 "" H 10000 2600 50  0001 C CNN
-	1    10000 2600
-	1    0    0    -1
+P 9900 2950
+F 0 "#PWR0142" H 9900 2800 50  0001 C CNN
+F 1 "+BATT" H 9915 3123 50  0000 C CNN
+F 2 "" H 9900 2950 50  0001 C CNN
+F 3 "" H 9900 2950 50  0001 C CNN
+	1    9900 2950
+	-1   0    0    1
 $EndComp
 $Comp
 L power:GND #PWR0143
 U 1 1 5CB481BB
-P 9850 3000
-F 0 "#PWR0143" H 9850 2750 50  0001 C CNN
-F 1 "GND" H 9855 2827 50  0000 C CNN
-F 2 "" H 9850 3000 50  0001 C CNN
-F 3 "" H 9850 3000 50  0001 C CNN
-	1    9850 3000
-	1    0    0    -1
+P 9900 2650
+F 0 "#PWR0143" H 9900 2400 50  0001 C CNN
+F 1 "GND" H 9905 2477 50  0000 C CNN
+F 2 "" H 9900 2650 50  0001 C CNN
+F 3 "" H 9900 2650 50  0001 C CNN
+	1    9900 2650
+	-1   0    0    1
 $EndComp
-Wire Wire Line
-	10150 2600 10000 2600
-Wire Wire Line
-	10150 2700 10000 2700
-Wire Wire Line
-	10000 2700 10000 2600
-Connection ~ 10000 2600
-Wire Wire Line
-	10150 2850 10000 2850
-Wire Wire Line
-	10000 2850 10000 2700
-Connection ~ 10000 2700
-Wire Wire Line
-	10150 2950 10000 2950
-Wire Wire Line
-	10000 2950 10000 2850
-Connection ~ 10000 2850
-Wire Wire Line
-	10150 2650 9850 2650
-Wire Wire Line
-	9850 2650 9850 2750
-Wire Wire Line
-	10150 2750 9850 2750
-Connection ~ 9850 2750
-Wire Wire Line
-	9850 2750 9850 2900
-Wire Wire Line
-	10150 2900 9850 2900
-Connection ~ 9850 2900
-Wire Wire Line
-	9850 2900 9850 3000
-Wire Wire Line
-	10150 3000 9850 3000
-Connection ~ 9850 3000
 $Comp
 L final_project-rescue:2_pin_screw_terminal U12
@@
 	1    0    0    -1
 $EndComp
+Wire Wire Line
+	10150 2600 10000 2600
+Wire Wire Line
+	10000 2600 10000 2700
+Wire Wire Line
+	10000 2700 10150 2700
+Wire Wire Line
+	10150 2900 10000 2900
+Wire Wire Line
+	10000 2900 10000 3000
+Wire Wire Line
+	10000 3000 10150 3000
+Wire Wire Line
+	10000 2900 10000 2700
+Connection ~ 10000 2900
+Connection ~ 10000 2700
+Wire Wire Line
+	10150 2650 9900 2650
+Wire Wire Line
+	9900 2650 9900 2750
+Wire Wire Line
+	9900 2750 10150 2750
+Connection ~ 9900 2650
+Wire Wire Line
+	10150 2850 9900 2850
+Wire Wire Line
+	9900 2850 9900 2950
+Wire Wire Line
+	9900 2950 10150 2950
+Connection ~ 9900 2950
 $EndSCHEMATC
