File: final_project/final_project.kicad_pcb (KiCad board)
At the start: 2 copper layers, 82.3 x 76.7 mm, 62 parts, among them J1 USB_microB_2040002-1, J2 Arduino_ICSP, J3 Conn_01x06_Male, U1 FT232RQ, U10 MAX14870, U11 TXB0108_DQS, U12 2_pin_screw_terminal, U13 8_pin_screw_terminal, U14 8_pin_screw_terminal, U2 MCP1702T-5002E_CB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

Commit message: updated layout v1
Parts:
- moved C13 2.70 mm to (182.3, 69.3)
- moved R17 2.55 mm to (169.9, 76.1)
- moved R18 2.55 mm to (166.1, 71.1)
- moved R19 2.55 mm to (182.4, 67.5)
- moved R20 2.55 mm to (182.5, 71.5)
- moved U5 2.55 mm to (169.6, 72.9)
- moved D6 2.55 mm to (166.4, 73.5)
- moved D8 2.55 mm to (182.9, 73.5)
- moved D5 2.54 mm to (169.8, 78.1), turned to 180 degrees
- moved D7 1.82 mm to (184.2, 65.3)
Connections:
- U13 pad 1: +BATT -> Net-(U13-Pad1)
- U13 pad 3: +BATT -> Net-(U13-Pad1)
- U13 pad 6: GND -> Net-(U13-Pad1)
- U13 pad 8: GND -> Net-(U13-Pad1)
Routing:
- net GND: track 171.3 -> 206.5 mm, vias 26 -> 29
- net Net-(U13-Pad1): track 0.00 -> 32.1 mm
- net +BATT: track 13.9 -> 29.1 mm, vias 0 -> 1
- net +3V3: track 111.9 -> 123.7 mm, vias 6 -> 7
- net /logic1_3: track 39.3 -> 43.6 mm
- net /logic4_3: track 27.5 -> 25.3 mm
- net /logic2_3: track 28.7 -> 26.6 mm
- net /logic3_3: track 27.8 -> 25.8 mm
- net Net-(R12-Pad1): track 12.6 -> 14.1 mm
- net /motor4b: track 15.6 -> 17.1 mm
- net Net-(R15-Pad1): track 10.5 -> 11.8 mm
- net +5V: track 79.8 -> 80.8 mm, vias 14 -> 16
- net /motor1a: track 16.0 -> 16.6 mm
Other:
- board size 82.3 x 76.7 mm -> 73 x 74 mm
- board text added: "1+"
- board text added: "1-"
- board text added: "2+"
- board text added: "2-"
- board text added: "3+"
- board text added: "3-"
- board text added: "4+"
- board text added: "4-"
- board text added: "ArdConn"
- board text added: "BATTERY"
- board text added: "BT PWR"
- board text added: "LowBatt"
- board text added: "MOTOR"
- board text added: "RF Actv"

Commit message: layout update
Parts:
- C13: value 1µF -> 10µF; footprint Capacitor_SMD:C_0603_1608Metric -> Capacitor_SMD:C_0805_2012Metric
- R17, R19, R20: value 1k -> 330
- moved C1 11.8 mm to (137.4, 107.7)
- moved C2 5.85 mm to (148.1, 112.5), turned to 180 degrees
- moved C3 3.57 mm to (145.3, 116.3)
- moved C10 2.18 mm to (147.9, 89.2), turned to 180 degrees
- moved C9 1.88 mm to (144.8, 88.7), turned to 270 degrees
- moved D5 1.82 mm to (169.4, 76.3), turned to 90 degrees
- moved R17 1.48 mm to (171.4, 76.2), turned to 90 degrees
- moved R20 0.75 mm to (182.7, 72.3)
- moved D8 0.62 mm to (182.9, 74.2)
- moved R19 0.39 mm to (182.2, 67.2)
Connections:
- D5 pad 2: +5V -> +3V3
- D7 pad 2: +5V -> +3V3
- D8 pad 2: +5V -> +3V3
Routing:
- net +5V: track 80.8 -> 45.3 mm, vias 16 -> 11
- net +3V3: track 123.7 -> 137.0 mm, vias 7 -> 8
- net GND: track 206.5 -> 216.4 mm, vias 29 -> 35
- net /logic1_5: track 22.7 -> 27.9 mm
- net /A6: track 86.4 -> 89.0 mm
- net /AREF: track 4.06 -> 1.68 mm
- net Net-(R3-Pad1): track 11.7 -> 13.9 mm
- net /logic6_5: track 19.2 -> 20.5 mm
- net /LowBatt: track 3.37 -> 2.58 mm
- net Net-(D5-Pad1): track 2.67 -> 2.12 mm
- added copper zone on B.Cu, net GND

Commit message: layout edit ground traces
Routing:
- net GND: track 216.4 -> 206.6 mm, vias 35 -> 38
- net /PowerOn: track 5.41 -> 6.73 mm
